File: KiCAD Files/RRIA_accelerometer.kicad_sch (KiCad schematic)
At the start: 15 parts, among them J2 SPI LIS3DH, M1 Logo_Duet3d_New, U1 LIS3DH

Commit message: gitignore + prep for RP2040
Parts:
- removed J2: SPI LIS3DH, Connector_IDC:IDC-Header_2x05_P2.54mm_Vertical, symbol Connector_Generic:Conn_02x05_Odd_Even
- removed M1: Logo_Duet3d_New, complib:LOGO_NEW_Duet3D_vertical_6mm_no_mask, symbol Duet3:Logo_Duet3d_New
- C21: renamed from C2; value 10u 10V -> 10u 10V
- renumbered C1 to C20, C3 to C23, C4 to C24
Connections:
- no-connect marks 6 -> 3
Other:
- moved on the sheet: C20, C21, C23, C24, D1, H1, R1, R2, R3, R4, R5, R6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

Commit message: progress
Parts:
- removed C23, C24: 470p 6.3V, Capacitor_SMD:C_0402_1005Metric_Wbry, symbol Device:C_Small
- removed D1: PWR, LED_SMD:LED_0603_1608Metric, symbol Device:LED
- removed H1: M6, MountingHole:MountingHole_6mm, symbol Mechanical:MountingHole
- removed R1, R2, R3, R4, R5: 62R, Resistor_SMD:R_0402_1005Metric_Wbry, symbol Device:R_Small
- removed R6: 220R, Resistor_SMD:R_0402_1005Metric_Wbry, symbol Device:R_Small
- added C1, C10, C15, C16, C19, C2, C25, C26, C3, C4, C5, C7, C8, C9: 100nF, Capacitor_SMD:C_0402_1005Metric, symbol Device:C_Small
- added C11, C12, C22, C27, C28, C6: 1uF, Capacitor_SMD:C_0402_1005Metric, symbol Device:C_Small
- added C13, C14: 10pF, Capacitor_SMD:C_0402_1005Metric, symbol Device:C_Small
- added C17, C18: 8pF, Capacitor_SMD:C_0402_1005Metric, symbol Device:C_Small
- added J3: 2.54-Header-1x2, Connector_PinHeader_2.54mm:PinHeader_1x02_P2.54mm_Vertical, symbol Connector_Generic:Conn_01x02
- added R10: 1k, Resistor_SMD:R_0402_1005Metric, symbol Device:R_Small
- added R7: 120Ω, PCM_Resistor_SMD_AKL:R_0402_1005Metric, symbol Device:R_Small
- added SW1, SW2: TS-1088, Button_Switch_SMD:SW_SPST_TS-1088-xR025, symbol Switch:SW_SPST
- added U2: RP2040, Package_DFN_QFN:QFN-56-1EP_7x7mm_P0.4mm_EP3.2x3.2mm_ThermalVias, symbol MCU_RaspberryPi:RP2040
- added U3: IS25WP016D, Package_SON:Winbond_USON-8-1EP_3x2mm_P0.5mm_EP0.2x1.6mm, symbol Memory_Flash:W25Q128JVS
- added U4: MCP2518FD-xQBB, PCM_Package_DFN_QFN_AKL:DFN-14-1EP_3x4.5mm_P0.65mm_EP1.65x4.25mm, symbol Interface_CAN_LIN:MCP2518FD-xQBB
- added U5: MCP2542FDxMF, PCM_Package_DFN_QFN_AKL:DFN-8-1EP_3x3mm_P0.65mm_EP1.7x2.05mm, symbol Interface_CAN_LIN:MCP2542FDxMF
- added Y1: 12MHz, Crystal:Crystal_SMD_2520-4Pin_2.5x2.0mm, symbol Device:Crystal_GND24
- added Y2: 40MHz, symbol Device:Crystal_GND24
- C20: value 0u1 6.3V -> 100nF; footprint Capacitor_SMD:C_0402_1005Metric_Wbry -> Capacitor_SMD:C_0402_1005Metric; LCSC (none) -> C541464; Part Number 1uF 6.3V X7R 0402 -> (none)
- C21: value 10u 10V -> 1uF; footprint Capacitor_SMD:C_0603_1608Metric_Wbry -> Capacitor_SMD:C_0402_1005Metric; LCSC (none) -> C2887020; Part Number 10u 10V 10% X7R -> (none)
Connections:
- net SCL is gone; now on net SPI_SCK: U1.4 (SCL/SPC)
- net SDI is gone; now on net SPI_MOSI: U1.6 (SDA/SDI)
- net SDO is gone; now on net SPI_MISO: U1.7 (SDO/SA0)
- net int1 is gone; now on net INT1: U1.11 (INT1)
- net GND: now also C20.1, C21.1, C1.1, C10.1, C11.1, C12.1, C13.1, C14.1, C15.1, C16.1, C17.1, C18.1, C19.2, C2.1, C22.2, C25.1, C26.2, C27.1, C28.2, C3.1, C4.1, C5.1, C6.1, C7.1, C8.1, C9.1, SW1.1 (A), SW2.1 (A), U2.19 (TESTEN), U2.57 (GND), U3.4 (GND), U3.9 (GND), U4.15 (VSS), U4.7 (VSS), U5.2 (VSS), U5.8 (STBY), U5.9 (VSS), Y1.2, Y1.4, Y2.2 (G), Y2.4 (G); no longer C20.2, C21.2
- net INT1: now also U2.11 (GPIO8)
- net SPI_MISO: now also U2.14 (GPIO11), U4.12 (SDO)
- net SPI_MOSI: now also U2.15 (GPIO12), U4.11 (SDI)
- net SPI_SCK: now also U2.13 (GPIO10), U4.10 (SCK)
- net 3.3V renamed +3V3
- net +3V3: now also C20.2, C21.2, C1.2, C10.2, C11.2, C12.2, C19.1, C2.2, C22.1, C26.1, C28.1, C3.2, C4.2, C5.2, C7.2, C8.2, C9.2, U2.1 (IOVDD), U2.10 (IOVDD), U2.22 (IOVDD), U2.33 (IOVDD), U2.42 (IOVDD), U2.43 (ADC_AVDD), U2.44 (VREG_IN), U2.48 (USB_VDD), U2.49 (IOVDD), U3.8 (VCC), U4.14 (VDD), U5.5 (VIO); no longer C20.1, C21.1
- net cs renamed CS_LIS
- net CS_LIS: now also U2.12 (GPIO9)
- new net: J3.2 (Pin_2), U5.6 (CANL)
- new net: R7.1, U5.7 (CANH)
- new net: J3.1 (Pin_1), R7.2
- new net: C14.2, R10.1, Y1.3
- new net +1V1: C15.2, C16.2, C6.2, U2.23 (DVDD), U2.45 (VREG_VOUT), U2.50 (DVDD)
- new net +5V: C25.2, C27.2, U5.3 (VDD)
- new net CAN-RX: U4.2 (RXCAN), U5.4 (RXD)
- new net CAN-TX: U4.1 (TXCAN), U5.1 (TXD)
- new net CS_CANFD: U2.17 (GPIO14), U4.13 (~{CS})
- new net MCP_INT: U2.16 (GPIO13), U4.4 (~{INT})
- new net OSC1: C18.2, U4.6 (OSC1), Y2.3
- new net OSC2: C17.2, U4.5 (OSC2), Y2.1
- new net QSPI-CLK: U2.52 (QSPI_SCLK), U3.6 (CLK)
- new net QSPI-SS: SW2.2 (B), U2.56 (QSPI_SS), U3.1 (~{CS})
- new net RUN: SW1.2 (B), U2.26 (RUN)
- new net SD0: U2.53 (QSPI_SD0), U3.5 (DI(IO0))
- new net SD1: U2.55 (QSPI_SD1), U3.2 (DO(IO1))
- new net SD2: U2.54 (QSPI_SD2), U3.3 (IO2)
- new net SD3: U2.51 (QSPI_SD3), U3.7 (IO3)
- new net USB_D+: U2.47 (USB_DP)
- new net USB_D-: U2.46 (USB_DM)
- new net XIN: C13.2, U2.20 (XIN), Y1.1
- new net XOUT: R10.2, U2.21 (XOUT)
- no-connect marks 3 -> 21
Other:
- note added: "12MHz CRYSTAL"
- note added: "2MB FLASH"
- note added: "CAN Convertor"
- note added: "MCP2518 Caps"
- note added: "MCP2542 Caps"
- note removed: "Duet3D Accelerometer"
- note removed: "SPI & Power"
- moved on the sheet: U1

Commit message: Final
Parts:
- added C23, C29: 1uF, Capacitor_SMD:C_0402_1005Metric, symbol Device:C_Small
- added C24, C30: 100nF, Capacitor_SMD:C_0402_1005Metric, symbol Device:C_Small
- added D1: GRN, PCM_LED_SMD_AKL:LED_0805_2012Metric, symbol Device:LED_Small
- added D2: RED, PCM_LED_SMD_AKL:LED_0805_2012Metric, symbol Device:LED_Small
- added J1: Conn_01x04, Connector_JST:JST_XH_S4B-XH-A_1x04_P2.50mm_Horizontal, symbol Connector_Generic:Conn_01x04
- added J2: USB_C_Receptacle_USB2.0_16P, CustomFootprints:USB_C_Receptacle_HRO_TYPE-C-31-M-12, symbol Connector:USB_C_Receptacle_USB2.0_16P
- added R1, R2: 5.1kΩ, PCM_Resistor_SMD_AKL:R_0402_1005Metric, symbol Device:R_Small
- added R3, R4: 1kΩ, PCM_Resistor_SMD_AKL:R_0402_1005Metric, symbol Device:R_Small
- added U6: TLV75733PDBV, PCM_Package_TO_SOT_SMD_AKL:SOT-23-5, symbol Regulator_Linear:TLV75733PDBV
- added U7: USBLC6-2SC6, PCM_Package_TO_SOT_SMD_AKL:SOT-23-6, symbol Power_Protection:USBLC6-2SC6
Connections:
- net +3V3: now also C29.2, C30.2, R3.1, U6.5 (OUT)
- net +5V: now also C23.2, C24.2, J1.1 (Pin_1), J2.A4 (VBUS), J2.A9 (VBUS), J2.B4 (VBUS), J2.B9 (VBUS), U6.1 (IN), U6.3 (EN), U7.5 (VBUS)
- net CANH: now also J3.2 (Pin_2), U5.6 (CANL), J1.2 (Pin_2)
- net CANL: now also R7.1, U5.7 (CANH), J1.3 (Pin_3)
- net GND: now also C23.1, C24.1, C29.1, C30.1, D1.1 (K), D2.1 (K), J1.4 (Pin_4), J2.A1 (GND), J2.A12 (GND), J2.B1 (GND), J2.B12 (GND), J2.S1 (SHIELD), R1.1, R2.1, U6.2 (GND), U7.2 (GND)
- net USB_D+: now also U7.4 (I/O2)
- net USB_D-: now also U7.6 (I/O1)
- new net: J2.A5 (CC1), R1.2
- new net: D1.2 (A), R3.2
- new net: D2.2 (A), R4.2
- new net: J2.B5 (CC2), R2.2
- new net: J2.A7 (D-), J2.B7 (D-), U7.1 (I/O1)
- new net: J2.A6 (D+), J2.B6 (D+), U7.3 (I/O2)
- new net LED: R4.1
- no-connect marks 21 -> 23
Other:
- note added: "USB Port"
- note removed: "MCP2542 Caps"
- moved on the sheet: C25, C26, C27, C28, J3, R7
